File: abbyWatchV1.kicad_pcb (KiCad board)
At the start: 4 copper layers, 40 x 35 mm, 69 parts, among them J1 Conn_01x02, J2 SJ-3524-SMT, Q1 2N7002, U1 BH1792GLC-E2, U10 XC6209, U11 MCP73831T-2ACI_OT, U13 XC6209, U15 TLA2022IRUGR, U16 LM324D, U2 BMA400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

Commit message: Added project images and all component CAD models
Parts:
- moved S2 0.13 mm to (92.8, 91.3)
- moved C15 0.08 mm to (63.8, 107.7)
Routing:
- net /VBUS: track 48.4 -> 49.3 mm
